File: prototype/filestick-prototype/filestick-prototype.kicad_sch (KiCad schematic)
At the start: 53 parts, among them J1 DIN-5, J2 DIN-5, J3 GPIO header 1, J4 UART header, J5 GPIO header 2, J6 SPI header, Q1 2N7002, Q2 2N7002, Q3 2N7002, Q4 2N7002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

Commit message: add capacitor to SD card IF
Parts:
- added C9: 100nF, Capacitor_SMD:C_0603_1608Metric_Pad1.08x0.95mm_HandSolder, symbol Device:C
Connections:
- net +3.3V: now also C9.1
- net GND: now also C9.2
Changed lines of the file:
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@@
   (junction (at 82.55 50.8) (diameter 0) (color 0 0 0 0)
   )
+  (junction (at 337.82 124.46) (diameter 0) (color 0 0 0 0)
+  )
   (junction (at 55.88 152.4) (diameter 0) (color 0 0 0 0)
   )
@@
   (junction (at 87.63 64.77) (diameter 0) (color 0 0 0 0)
   )
-  (junction (at 337.82 130.81) (diameter 0) (color 0 0 0 0)
+  (junction (at 327.66 135.89) (diameter 0) (color 0 0 0 0)
   )
   (junction (at 48.26 35.56) (diameter 0) (color 0 0 0 0)
@@
   )
   (junction (at 107.95 180.34) (diameter 0) (color 0 0 0 0)
+  )
+  (junction (at 327.66 124.46) (diameter 0) (color 0 0 0 0)
   )
   (junction (at 33.02 77.47) (diameter 0) (color 0 0 0 0)
@@
     (stroke (width 0) (type default) (color 0 0 0 0))
   )
-  (wire (pts (xy 337.82 135.89) (xy 322.58 135.89))
+  (wire (pts (xy 337.82 135.89) (xy 327.66 135.89))
     (stroke (width 0) (type default) (color 0 0 0 0))
   )
@@
     (stroke (width 0) (type default) (color 0 0 0 0))
   )
-  (wire (pts (xy 337.82 130.81) (xy 320.04 130.81))
+  (wire (pts (xy 337.82 124.46) (xy 327.66 124.46))
     (stroke (width 0) (type default) (color 0 0 0 0))
   )
@@
     (stroke (width 0) (type default) (color 0 0 0 0))
   )
+  (wire (pts (xy 327.66 124.46) (xy 320.04 124.46))
+    (stroke (width 0) (type default) (color 0 0 0 0))
+  )
   (wire (pts (xy 57.15 175.26) (xy 72.39 175.26))
     (stroke (width 0) (type default) (color 0 0 0 0))
@@
     (stroke (width 0) (type default) (color 0 0 0 0))
   )
+  (wire (pts (xy 327.66 133.35) (xy 327.66 135.89))
+    (stroke (width 0) (type default) (color 0 0 0 0))
+  )
   (wire (pts (xy 295.91 226.06) (xy 318.77 226.06))
     (stroke (width 0) (type default) (color 0 0 0 0))
@@
     (stroke (width 0) (type default) (color 0 0 0 0))
   )
-  (wire (pts (xy 358.14 156.21) (xy 358.14 130.81))
+  (wire (pts (xy 358.14 156.21) (xy 358.14 124.46))
     (stroke (width 0) (type default) (color 0 0 0 0))
   )
@@
     (stroke (width 0) (type default) (color 0 0 0 0))
   )
-  (wire (pts (xy 320.04 130.81) (xy 320.04 152.4))
+  (wire (pts (xy 320.04 124.46) (xy 320.04 152.4))
     (stroke (width 0) (type default) (color 0 0 0 0))
   )
@@
     (stroke (width 0) (type default) (color 0 0 0 0))
   )
+  (wire (pts (xy 327.66 124.46) (xy 327.66 125.73))
+    (stroke (width 0) (type default) (color 0 0 0 0))
+  )
   (wire (pts (xy 204.47 194.31) (xy 204.47 193.04))
     (stroke (width 0) (type default) (color 0 0 0 0))
@@
     (stroke (width 0) (type default) (color 0 0 0 0))
   )
+  (wire (pts (xy 327.66 135.89) (xy 322.58 135.89))
+    (stroke (width 0) (type default) (color 0 0 0 0))
+  )
   (wire (pts (xy 243.84 158.75) (xy 250.19 158.75))
     (stroke (width 0) (type default) (color 0 0 0 0))
   )
-  (wire (pts (xy 358.14 130.81) (xy 337.82 130.81))
+  (wire (pts (xy 358.14 124.46) (xy 337.82 124.46))
     (stroke (width 0) (type default) (color 0 0 0 0))
   )
@@
     (pin "2")
   )
-  (symbol (lib_id "power:+3.3V") (at 337.82 130.81 0) (unit 1)
-    (in_bom yes) (on_board yes) (fields_autoplaced)
-    (property "Reference" "#PWR026" (id 0) (at 337.82 134.62 0)
-      (effects (font (size 1.27 1.27)) hide)
-    )
-    (property "Value" "+3.3V" (id 1) (at 337.82 125.73 0))
-    (property "Footprint" "" (id 2) (at 337.82 130.81 0)
-      (effects (font (size 1.27 1.27)) hide)
-    )
-    (property "Datasheet" "" (id 3) (at 337.82 130.81 0)
+  (symbol (lib_id "power:+3.3V") (at 337.82 124.46 0) (unit 1)
+    (in_bom yes) (on_board yes) (fields_autoplaced)
+    (property "Reference" "#PWR026" (id 0) (at 337.82 128.27 0)
+      (effects (font (size 1.27 1.27)) hide)
+    )
+    (property "Value" "+3.3V" (id 1) (at 337.82 119.38 0))
+    (property "Footprint" "" (id 2) (at 337.82 124.46 0)
+      (effects (font (size 1.27 1.27)) hide)
+    )
+    (property "Datasheet" "" (id 3) (at 337.82 124.46 0)
       (effects (font (size 1.27 1.27)) hide)
     )
@@
     (pin "1")
   )
+  (symbol (lib_id "Device:C") (at 327.66 129.54 0) (unit 1)
+    (in_bom yes) (on_board yes) (fields_autoplaced)
+    (property "Reference" "C9" (id 0) (at 331.47 128.2699 0)
+      (effects (font (size 1.27 1.27)) (justify left))
+    )
+    (property "Value" "100nF" (id 1) (at 331.47 130.8099 0)
+      (effects (font (size 1.27 1.27)) (justify left))
+    )
+    (property "Footprint" "Capacitor_SMD:C_0603_1608Metric_Pad1.08x0.95mm_HandSolder" (id 2) (at 328.6252 133.35 0)
+      (effects (font (size 1.27 1.27)) hide)
+    )
+    (property "Datasheet" "~" (id 3) (at 327.66 129.54 0)
+      (effects (font (size 1.27 1.27)) hide)
+    )
+    (pin "1")
+    (pin "2")
+  )
   (symbol (lib_id "Device:R") (at 308.61 53.34 0) (unit 1)
     (in_bom yes) (on_board yes) (fields_autoplaced)
@@
       (reference "C8") (unit 1) (value "100nF") (footprint "Capacitor_SMD:C_0603_1608Metric_Pad1.08x0.95mm_HandSolder")
     )
+    (path "/bb4253f1-a91b-4c7e-8fe9-5a850aa91259"
+      (reference "C9") (unit 1) (value "100nF") (footprint "Capacitor_SMD:C_0603_1608Metric_Pad1.08x0.95mm_HandSolder")
+    )
     (path "/3354a6fc-63a3-43be-ab16-343a45076103"

Commit message: PCB and footprints
Parts:
- U2: footprint Package_SO:SOIC-14_3.9x8.7mm_P1.27mm -> Package_SO:SO-14_5.3x10.2mm_P1.27mm
- U4: footprint Package_DIP:DIP-48_W15.24mm_Socket -> filestick-footprints:DIP48_0.7in
Changed lines of the file:
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@@
       (effects (font (size 1.27 1.27)) (justify left))
     )
-    (property "Footprint" "Package_DIP:DIP-48_W15.24mm_Socket" (id 2) (at 274.32 143.51 0)
+    (property "Footprint" "filestick-footprints:DIP48_0.7in" (id 2) (at 274.32 143.51 0)
       (effects (font (size 1.27 1.27)) hide)
     )
@@
     (property "Reference" "U2" (id 0) (at 267.97 43.18 0))
     (property "Value" "LMV324" (id 1) (at 269.24 50.8 0))
-    (property "Footprint" "Package_SO:SOIC-14_3.9x8.7mm_P1.27mm" (id 2) (at 264.16 49.53 0)
+    (property "Footprint" "Package_SO:SO-14_5.3x10.2mm_P1.27mm" (id 2) (at 264.16 49.53 0)
       (effects (font (size 1.27 1.27)) hide)
     )
@@
       (effects (font (size 1.27 1.27)) (justify left))
     )
-    (property "Footprint" "Package_SO:SOIC-14_3.9x8.7mm_P1.27mm" (id 2) (at 76.2 232.41 0)
+    (property "Footprint" "Package_SO:SO-14_5.3x10.2mm_P1.27mm" (id 2) (at 76.2 232.41 0)
       (effects (font (size 1.27 1.27)) hide)
     )
@@
     (property "Reference" "U2" (id 0) (at 80.01 209.55 0))
     (property "Value" "LMV324" (id 1) (at 81.28 217.17 0))
-    (property "Footprint" "Package_SO:SOIC-14_3.9x8.7mm_P1.27mm" (id 2) (at 76.2 215.9 0)
+    (property "Footprint" "Package_SO:SO-14_5.3x10.2mm_P1.27mm" (id 2) (at 76.2 215.9 0)
       (effects (font (size 1.27 1.27)) hide)
     )
@@
     (property "Reference" "U2" (id 0) (at 80.01 231.14 0))
     (property "Value" "LMV324" (id 1) (at 81.28 238.76 0))
-    (property "Footprint" "Package_SO:SOIC-14_3.9x8.7mm_P1.27mm" (id 2) (at 76.2 237.49 0)
+    (property "Footprint" "Package_SO:SO-14_5.3x10.2mm_P1.27mm" (id 2) (at 76.2 237.49 0)
       (effects (font (size 1.27 1.27)) hide)
     )
@@
     (property "Reference" "U2" (id 0) (at 264.16 62.23 0))
     (property "Value" "LMV324" (id 1) (at 275.59 71.12 0))
-    (property "Footprint" "Package_SO:SOIC-14_3.9x8.7mm_P1.27mm" (id 2) (at 266.7 68.58 0)
+    (property "Footprint" "Package_SO:SO-14_5.3x10.2mm_P1.27mm" (id 2) (at 266.7 68.58 0)
       (effects (font (size 1.27 1.27)) hide)
     )
@@
     )
     (path "/b19894d5-7fa9-4eca-8f7f-504f876287db"
-      (reference "U2") (unit 1) (value "LMV324") (footprint "Package_SO:SOIC-14_3.9x8.7mm_P1.27mm")
+      (reference "U2") (unit 1) (value "LMV324") (footprint "Package_SO:SO-14_5.3x10.2mm_P1.27mm")
     )
     (path "/c8d9109f-29ec-4dcc-8afa-923b80be6987"
-      (reference "U2") (unit 2) (value "LMV324") (footprint "Package_SO:SOIC-14_3.9x8.7mm_P1.27mm")
+      (reference "U2") (unit 2) (value "LMV324") (footprint "Package_SO:SO-14_5.3x10.2mm_P1.27mm")
     )
     (path "/32f44d8e-aa46-4c1f-b9ba-55ec78a09e8c"
-      (reference "U2") (unit 3) (value "LMV324") (footprint "Package_SO:SOIC-14_3.9x8.7mm_P1.27mm")
+      (reference "U2") (unit 3) (value "LMV324") (footprint "Package_SO:SO-14_5.3x10.2mm_P1.27mm")
     )
     (path "/b06ce78a-852b-4fdf-ad38-fd7516f708ba"
-      (reference "U2") (unit 4) (value "LMV324") (footprint "Package_SO:SOIC-14_3.9x8.7mm_P1.27mm")
+      (reference "U2") (unit 4) (value "LMV324") (footprint "Package_SO:SO-14_5.3x10.2mm_P1.27mm")
     )
     (path "/47163286-6007-4ebb-9ba0-6b76e2eec328"
-      (reference "U2") (unit 5) (value "LMV324") (footprint "Package_SO:SOIC-14_3.9x8.7mm_P1.27mm")
+      (reference "U2") (unit 5) (value "LMV324") (footprint "Package_SO:SO-14_5.3x10.2mm_P1.27mm")
     )
     (path "/729fac80-7f4c-4077-9d0c-4f5f4f39b6ed"
@@
     )
     (path "/0a57b3fc-b5d8-489f-8f4c-c5c0980bca2c"
-      (reference "U4") (unit 1) (value "Upduino 3.1") (footprint "Package_DIP:DIP-48_W15.24mm_Socket")
+      (reference "U4") (unit 1) (value "Upduino 3.1") (footprint "filestick-footprints:DIP48_0.7in")
     )
     (path "/92a70b4c-5f05-47f9-938a-facc779a7322"

Commit message: clamp collision detection at 3v3, add leds etc
Parts:
- added D4: D_Zener 3.3v, Diode_SMD:D_SOD-323_HandSoldering, symbol Device:D_Zener
- added D5, D6: LED, LED_SMD:LED_0603_1608Metric_Pad1.05x0.95mm_HandSolder, symbol Device:LED
- added R18: 1k, Resistor_SMD:R_0603_1608Metric_Pad0.98x0.95mm_HandSolder, symbol Device:R
- added R19, R20: 560, Resistor_SMD:R_0603_1608Metric_Pad0.98x0.95mm_HandSolder, symbol Device:R
- SW1: footprint Button_Switch_THT:SW_PUSH_6mm -> Button_Switch_SMD:SW_Push_1P1T_NO_6x6mm_H9.5mm
Connections:
- net COLLISION_DETECT: now also D4.2 (A), R18.1; no longer U2.7
- net ECONET_CLKEN: now also R19.1
- net GND: now also D5.1 (K), D6.1 (K), R18.2
- net TERM_EN: now also R20.1
- new net: D5.2 (A), R19.2
- new net: D6.2 (A), R20.2
- new net COLLISION_DETECT_5V: D4.1 (K), U2.7

Commit message: better level shifter
Parts:
- removed D4: D_Zener 3.3v, Diode_SMD:D_SOD-323_HandSoldering, symbol Device:D_Zener
- added Q?: 2N7002, Package_TO_SOT_SMD:SOT-23, symbol Transistor_FET:2N7002
Connections:
- net +3.3V: now also R18.1
- net COLLISION_DETECT: now also R18.2, Q?.3 (D); no longer R18.1
- net COLLISION_DETECT_5V: now also Q?.1 (G)
- net GND: now also Q?.2 (S); no longer R18.2
Other:
- moved on the sheet: R18
Changed lines of the file:
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@@
   (junction (at 276.86 46.99) (diameter 0) (color 0 0 0 0)
   )
-  (junction (at 246.38 76.2) (diameter 0) (color 0 0 0 0)
-  )
   (junction (at 308.61 46.99) (diameter 0) (color 0 0 0 0)
   )
@@
   (junction (at 63.5 255.27) (diameter 0) (color 0 0 0 0)
   )
+  (junction (at 233.68 90.17) (diameter 0) (color 0 0 0 0)
+  )
   (junction (at 241.3 26.67) (diameter 0) (color 0 0 0 0)
   )
@@
     (stroke (width 0) (type default) (color 0 0 0 0))
   )
+  (wire (pts (xy 241.3 97.79) (xy 246.38 97.79))
+    (stroke (width 0) (type default) (color 0 0 0 0))
+  )
   (wire (pts (xy 81.28 152.4) (xy 68.58 152.4))
     (stroke (width 0) (type default) (color 0 0 0 0))
@@
     (stroke (width 0) (type default) (color 0 0 0 0))
   )
-  (wire (pts (xy 226.06 76.2) (xy 246.38 76.2))
+  (wire (pts (xy 213.36 90.17) (xy 233.68 90.17))
     (stroke (width 0) (type default) (color 0 0 0 0))
   )
@@
     (stroke (width 0) (type default) (color 0 0 0 0))
   )
+  (wire (pts (xy 233.68 87.63) (xy 233.68 90.17))
+    (stroke (width 0) (type default) (color 0 0 0 0))
+  )
   (wire (pts (xy 365.76 172.72) (xy 363.22 172.72))
     (stroke (width 0) (type default) (color 0 0 0 0))
@@
     (stroke (width 0) (type default) (color 0 0 0 0))
   )
-  (wire (pts (xy 246.38 86.36) (xy 246.38 87.63))
-    (stroke (width 0) (type default) (color 0 0 0 0))
-  )
   (wire (pts (xy 48.26 58.42) (xy 48.26 55.88))
     (stroke (width 0) (type default) (color 0 0 0 0))
@@
     (stroke (width 0) (type default) (color 0 0 0 0))
   )
+  (wire (pts (xy 233.68 90.17) (xy 233.68 92.71))
+    (stroke (width 0) (type default) (color 0 0 0 0))
+  )
   (wire (pts (xy 355.6 175.26) (xy 365.76 175.26))
     (stroke (width 0) (type default) (color 0 0 0 0))
@@
     (stroke (width 0) (type default) (color 0 0 0 0))
   )
-  (wire (pts (xy 246.38 76.2) (xy 246.38 78.74))
-    (stroke (width 0) (type default) (color 0 0 0 0))
-  )
   (wire (pts (xy 241.3 26.67) (xy 243.84 26.67))
     (stroke (width 0) (type default) (color 0 0 0 0))
@@
     (stroke (width 0) (type default) (color 0 0 0 0))
   )
-  (wire (pts (xy 246.38 66.04) (xy 246.38 68.58))
+  (wire (pts (xy 246.38 66.04) (xy 246.38 97.79))
     (stroke (width 0) (type default) (color 0 0 0 0))
   )
@@
     (effects (font (size 1.27 1.27)) (justify left bottom))
   )
-  (label "COLLISION_DETECT" (at 226.06 76.2 0)
+  (label "COLLISION_DETECT" (at 213.36 90.17 0)
     (effects (font (size 1.27 1.27)) (justify left bottom))
   )
@@
     (pin "1")
   )
-  (symbol (lib_id "power:GND") (at 246.38 87.63 0) (unit 1)
+  (symbol (lib_id "power:GND") (at 233.68 102.87 0) (unit 1)
     (in_bom yes) (on_board yes) (fields_autoplaced)
-    (property "Reference" "#PWR0101" (id 0) (at 246.38 93.98 0)
+    (property "Reference" "#PWR0101" (id 0) (at 233.68 109.22 0)
       (effects (font (size 1.27 1.27)) hide)
     )
-    (property "Value" "GND" (id 1) (at 246.38 92.71 0))
-    (property "Footprint" "" (id 2) (at 246.38 87.63 0)
+    (property "Value" "GND" (id 1) (at 233.68 107.95 0))
+    (property "Footprint" "" (id 2) (at 233.68 102.87 0)
       (effects (font (size 1.27 1.27)) hide)
     )
-    (property "Datasheet" "" (id 3) (at 246.38 87.63 0)
+    (property "Datasheet" "" (id 3) (at 233.68 102.87 0)
       (effects (font (size 1.27 1.27)) hide)
     )
@@
     (pin "4")
   )
+  (symbol (lib_id "power:+3.3V") (at 233.68 80.01 0) (unit 1)
+    (in_bom yes) (on_board yes) (fields_autoplaced)
+    (property "Reference" "#PWR?" (id 0) (at 233.68 83.82 0)
+      (effects (font (size 1.27 1.27)) hide)
+    )
+    (property "Value" "+3.3V" (id 1) (at 233.68 74.93 0))
+    (property "Footprint" "" (id 2) (at 233.68 80.01 0)
+      (effects (font (size 1.27 1.27)) hide)
+    )
+    (property "Datasheet" "" (id 3) (at 233.68 80.01 0)
+      (effects (font (size 1.27 1.27)) hide)
+    )
+    (pin "1")
+  )
   (symbol (lib_id "power:GND") (at 364.49 196.85 0) (unit 1)
     (in_bom yes) (on_board yes) (fields_autoplaced)
@@
     (pin "1")
   )
-  (symbol (lib_id "Device:D_Zener") (at 246.38 72.39 270) (unit 1)
-    (in_bom yes) (on_board yes) (fields_autoplaced)
-    (property "Reference" "D4" (id 0) (at 248.92 71.1199 90)
-      (effects (font (size 1.27 1.27)) (justify left))
-    )
-    (property "Value" "D_Zener 3.3v" (id 1) (at 248.92 73.6599 90)
-      (effects (font (size 1.27 1.27)) (justify left))
-    )
-    (property "Footprint" "Diode_SMD:D_SOD-323_HandSoldering" (id 2) (at 246.38 72.39 0)
-      (effects (font (size 1.27 1.27)) hide)
-    )
-    (property "Datasheet" "~" (id 3) (at 246.38 72.39 0)
-      (effects (font (size 1.27 1.27)) hide)
-    )
-    (pin "1")
-    (pin "2")
-  )
   (symbol (lib_id "power:+3.3V") (at 227.33 25.4 0) (unit 1)
     (in_bom yes) (on_board yes) (fields_autoplaced)
@@
     (pin "1")
   )
+  (symbol (lib_id "Transistor_FET:2N7002") (at 236.22 97.79 0) (mirror y) (unit 1)
+    (in_bom yes) (on_board yes) (fields_autoplaced)
+    (property "Reference" "Q?" (id 0) (at 229.87 96.5199 0)
+      (effects (font (size 1.27 1.27)) (justify left))
+    )
+    (property "Value" "2N7002" (id 1) (at 229.87 99.0599 0)
+      (effects (font (size 1.27 1.27)) (justify left))
+    )
+    (property "Footprint" "Package_TO_SOT_SMD:SOT-23" (id 2) (at 231.14 99.695 0)
+      (effects (font (size 1.27 1.27) italic) (justify left) hide)
+    )
+    (property "Datasheet" "https://www.onsemi.com/pub/Collateral/NDS7002A-D.PDF" (id 3) (at 236.22 97.79 0)
+      (effects (font (size 1.27 1.27)) (justify left) hide)
+    )
+    (pin "1")
+    (pin "2")
+    (pin "3")
+  )
   (symbol (lib_id "Device:R") (at 139.7 213.36 90) (unit 1)
     (in_bom yes) (on_board yes) (fields_autoplaced)
@@
     (pin "1")
   )
-  (symbol (lib_id "Device:R") (at 246.38 82.55 0) (unit 1)
+  (symbol (lib_id "Device:R") (at 233.68 83.82 0) (unit 1)
     (in_bom yes) (on_board yes) (fields_autoplaced)
-    (property "Reference" "R18" (id 0) (at 248.92 81.2799 0)
+    (property "Reference" "R18" (id 0) (at 236.22 82.5499 0)
       (effects (font (size 1.27 1.27)) (justify left))
     )
-    (property "Value" "1k" (id 1) (at 248.92 83.8199 0)
+    (property "Value" "1k" (id 1) (at 236.22 85.0899 0)
       (effects (font (size 1.27 1.27)) (justify left))
     )
-    (property "Footprint" "Resistor_SMD:R_0603_1608Metric_Pad0.98x0.95mm_HandSolder" (id 2) (at 244.602 82.55 90)
+    (property "Footprint" "Resistor_SMD:R_0603_1608Metric_Pad0.98x0.95mm_HandSolder" (id 2) (at 231.902 83.82 90)
       (effects (font (size 1.27 1.27)) hide)
     )
-    (property "Datasheet" "~" (id 3) (at 246.38 82.55 0)
+    (property "Datasheet" "~" (id 3) (at 233.68 83.82 0)
       (effects (font (size 1.27 1.27)) hide)
     )
@@
       (reference "#PWR0101") (unit 1) (value "GND") (footprint "")
     )
+    (path "/4fa48868-af46-4293-be22-ae8095005663"
+      (reference "#PWR?") (unit 1) (value "+3.3V") (footprint "")
+    )
     (path "/1d828a71-404c-49c6-8956-820fdda0224a"
       (reference "#V0101") (unit 1) (value "VDD_TX") (footprint "")
@@
       (reference "D3") (unit 1) (value "BAT54S") (footprint "Package_TO_SOT_SMD:SOT-23")
     )
-    (path "/8aeb6658-d0a4-4065-b079-4e6cee32cd2a"
-      (reference "D4") (unit 1) (value "D_Zener 3.3v") (footprint "Diode_SMD:D_SOD-323_HandSoldering")
-    )
     (path "/23da723e-8f18-4153-9511-ef81ce62b89d"
       (reference "D5") (unit 1) (value "LED") (footprint "LED_SMD:LED_0603_1608Metric_Pad1.05x0.95mm_HandSolder")
@@
       (reference "Q4") (unit 1) (value "2N7002") (footprint "Package_TO_SOT_SMD:SOT-23")
     )
+    (path "/a435be7c-2bfb-4409-8c19-29abd1496700"
+      (reference "Q?") (unit 1) (value "2N7002") (footprint "Package_TO_SOT_SMD:SOT-23")
+    )
     (path "/132b8b80-d5dd-45a7-bb02-da5c00177cdf"

Commit message: Some unsaved stuff
Parts:
- gave numbers to parts that had none: 1
Changed lines of the file:
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@@
   (symbol (lib_id "power:+3.3V") (at 233.68 80.01 0) (unit 1)
     (in_bom yes) (on_board yes) (fields_autoplaced)
-    (property "Reference" "#PWR?" (id 0) (at 233.68 83.82 0)
+    (property "Reference" "#PWR0102" (id 0) (at 233.68 83.82 0)
       (effects (font (size 1.27 1.27)) hide)
     )
@@
   (symbol (lib_id "Transistor_FET:2N7002") (at 236.22 97.79 0) (mirror y) (unit 1)
     (in_bom yes) (on_board yes) (fields_autoplaced)
-    (property "Reference" "Q?" (id 0) (at 229.87 96.5199 0)
+    (property "Reference" "Q5" (id 0) (at 229.87 96.5199 0)
       (effects (font (size 1.27 1.27)) (justify left))
     )
@@
     )
     (path "/4fa48868-af46-4293-be22-ae8095005663"
-      (reference "#PWR?") (unit 1) (value "+3.3V") (footprint "")
+      (reference "#PWR0102") (unit 1) (value "+3.3V") (footprint "")
     )
     (path "/1d828a71-404c-49c6-8956-820fdda0224a"
@@
     )
     (path "/a435be7c-2bfb-4409-8c19-29abd1496700"
-      (reference "Q?") (unit 1) (value "2N7002") (footprint "Package_TO_SOT_SMD:SOT-23")
+      (reference "Q5") (unit 1) (value "2N7002") (footprint "Package_TO_SOT_SMD:SOT-23")
     )
     (path "/132b8b80-d5dd-45a7-bb02-da5c00177cdf"
