File: pcb/filestick/filestick.kicad_sch (KiCad schematic)
At the start: 96 parts

Commit message: Mainly add SD card to schematic
Parts:
- added C? (x2): C, symbol Device:C
- added C? (x2): 100nF, symbol Device:C
- added C? (x2): 4.7uF, symbol Device:C
- added D?: LED, symbol Device:LED
- added J?: Micro_SD_Card_Det, symbol Connector:Micro_SD_Card_Det
- added R?: 10k, symbol Device:R
- added R?: 560, symbol Device:R
- added R?: 1k, symbol Device:R
Connections:
- net FLASH_SS is gone; now on net FLASH_CS: U?.16 (IOB_35b_SPI_SS)
- net +3.3V: now also U?.1 (VCCIO_2), U?.33 (VCCIO_0), C?.1, C?.1, C?.2, C?.2, C?.2, C?.2, J?.4 (VDD), R?.1, R?.2
- net GND: now also J?.6 (Shield), C?.1, C?.1, C?.1, C?.1, C?.2, C?.2, D?.1 (K), J?.11 (SHIELD), J?.6 (VSS), J?.9 (DET_B)
- net at U?.7 (CDONE): now also R?.1
- net /CRESET: now reaches U?.8 (~{CRESET})
- net /CRESET: now also R?.2
- new net: D?.2 (A), R?.2
- new net SD_CS: J?.2 (DAT3/CD)
- new net SD_MISO: J?.7 (DAT0)
- new net SD_MOSI: J?.3 (CMD)
- new net SD_SCK: J?.5 (CLK)
- new net /SD_DETECT: J?.10 (DET_A), R?.1
- no-connect marks 1 -> 4
Other:
- note added: "MicroSD card"
- moved on the sheet: J?, U?A

Commit message: Finish schematic connections
Parts:
- removed J? (x2): DIN-5, filestick-footprints:Lumberg_DIN41524_5pin, symbol Connector:DIN-5
- removed TP?: Term En V TP, Connector_PinHeader_2.54mm:PinHeader_1x01_P2.54mm_Vertical, symbol Connector:Conn_01x01_Female
- removed TP?: Collision Mon TP, Connector_PinHeader_2.54mm:PinHeader_1x01_P2.54mm_Vertical, symbol Connector:Conn_01x01_Female
- removed TP?: VDD TX TP, Connector_PinHeader_2.54mm:PinHeader_1x01_P2.54mm_Vertical, symbol Connector:Conn_01x01_Female
- added J2, J3: DIN-5_180degree, symbol Connector:DIN-5_180degree
- added J5: Conn_01x08_Pin, symbol Connector:Conn_01x08_Pin
- added J6: Conn_01x09_Pin, symbol Connector:Conn_01x09_Pin
- added J7, J9: Conn_01x02_Pin, symbol Connector:Conn_01x02_Pin
- added J8: Conn_02x08_Odd_Even, symbol Connector_Generic:Conn_02x08_Odd_Even
- added TP1: VDD TX TP, symbol Connector:Conn_01x01_Socket
- added TP2: Collision Mon TP, symbol Connector:Conn_01x01_Socket
- added TP3: Term En 9V TP, symbol Connector:Conn_01x01_Socket
- gave numbers to parts that had none: 95
Connections:
- net +3.3V is gone; now on net +3V3: C10.2, C11.1, C12.2, C25.1, C26.1, C29.1, C6.2, C7.2, C8.2, C9.2, D9.1 (A), J4.4 (VDD), R1.1, R17.1, R18.1, R29.2, R5.2, R6.2, U1.1 (VCCIO_2), U1.22 (SPI_VCCIO1), U1.33 (VCCIO_0), U2.11 (~{RESET}), U4.8 (Vcc), U8.10 (+)
- net +3V3: now also J5.7 (Pin_7), J6.8 (Pin_8), J8.15 (Pin_15)
- net +5V: now also J8.13 (Pin_13)
- net CLK+: now also J2.5, J3.5
- net CLK-: now also J2.3, J3.3
- net COLLISION_MON: now also TP2.1 (Pin_1)
- net DATA+: now also J2.1, J3.4
- net DATA-: now also J2.4, J3.1
- net FLASH_CS: now also R11.2, J5.3 (Pin_3); no longer R12.2
- net FLASH_MISO: now also J5.4 (Pin_4)
- net FLASH_MOSI: now also J5.5 (Pin_5)
- net FLASH_SCK: now also R12.2, J5.6 (Pin_6); no longer R11.2
- net GND: now also J2.2, J3.2, J5.8 (Pin_8), J6.9 (Pin_9), J8.14 (Pin_14), J8.16 (Pin_16)
- net SD_CS: now also U1.48 (IOB_4a), J6.1 (Pin_1)
- net SD_MISO: now also U1.45 (IOB_5b), J6.4 (Pin_4)
- net SD_MOSI: now also U1.47 (IOB_2a), J6.2 (Pin_2)
- net SD_SCK: now also U1.46 (IOB_0a), J6.3 (Pin_3)
- net TERM_EN_9V: now also TP3.1 (Pin_1)
- net UART_RX: now also U1.25 (IOT_36b)
- net UART_TX: now also U1.23 (IOT_37a)
- net VDD_TX: now also TP1.1 (Pin_1)
- net /CRESET: now also J5.1 (Pin_1)
- net /SD_DETECT: now also U1.2 (IOB_6a), J6.5 (Pin_5)
- net GPIO_26: now reaches U1.26 (IOT_39a)
- net GPIO_26: now also J8.10 (Pin_10)
- net GPIO_37: now reaches U1.37 (IOT_45a_G1)
- net GPIO_37: now also J8.11 (Pin_11)
- net +2V5: now reaches C21.1, D8.1 (K), U1.24 (VPP_2V5)
- net UART_CBUS0: now reaches U2.15 (CBUS0)
- net UART_CBUS0: now also J7.1 (Pin_1)
- net UART_CBUS3: now reaches U2.16 (CBUS3)
- net UART_CBUS3: now also J7.2 (Pin_2)
- net UART_RTS: now reaches U2.2 (~{RTS})
- net UART_RTS: now also J9.2 (Pin_2)
- net UART_CTS: now reaches U2.6 (~{CTS})
- net UART_CTS: now also J9.1 (Pin_1)
- net GPIO_10: now reaches U1.10 (IOB_18a)
- net GPIO_10: now also J8.3 (Pin_3)
- net GPIO_11: now reaches U1.11 (IOB_20a)
- net GPIO_11: now also J8.4 (Pin_4)
- net GPIO_12: now reaches U1.12 (IOB_22a)
- net GPIO_12: now also J8.5 (Pin_5)
- net GPIO_13: now reaches U1.13 (IOB_24a)
- net GPIO_13: now also J8.6 (Pin_6)
- net GPIO_18: now reaches U1.18 (IOB_31b)
- net GPIO_18: now also J8.7 (Pin_7)
- net GPIO_19: now reaches U1.19 (IOB_29b)
- net GPIO_19: now also J8.8 (Pin_8)
- net GPIO_21: now reaches U1.21 (IOB_23b)
- net GPIO_21: now also J8.9 (Pin_9)
- net GPIO_6: now reaches U1.6 (IOB_13b)
- net GPIO_6: now also J8.1 (Pin_1)
- net CDONE: now reaches R4.1, U1.7 (CDONE)
- net CDONE: now also J5.2 (Pin_2)
- net GPIO_9: now reaches U1.9 (IOB_16a)
- net GPIO_9: now also J8.2 (Pin_2)
- net SPI_SS1: now reaches U1.3 (IOB_9b)
- net SPI_SS1: now also J6.6 (Pin_6)
- net SPI_SS2: now reaches U1.4 (IOB_8a)
- net SPI_SS2: now also J6.7 (Pin_7)
- net GPIO_44: now reaches U1.44 (IOB_3b_G6)
- net GPIO_44: now also J8.12 (Pin_12)
Other:
- note added: "GPIO Connector"
- moved on the sheet: C1, C10, C11, C12, C13, C14, C15, C17, C18, C19, C2, C20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

Commit message: Add footprints to schematic
Parts:
- removed J4: Micro_SD_Card_Det, symbol Connector:Micro_SD_Card_Det
- added J4: Micro_SD_Card_Det2, Connector_Card:microSD_HC_Hirose_DM3D-SF, symbol Connector:Micro_SD_Card_Det2
- added R35: 0, Resistor_SMD:R_0603_1608Metric_Pad0.98x0.95mm_HandSolder, symbol Device:R
- C1, C10, C12, C2, C23, C24, C3, C4, C5, C6, C7, C8, C9: footprint (none) -> Capacitor_SMD:C_0603_1608Metric_Pad1.08x0.95mm_HandSolder
- C25, C29: value C -> 100nF; footprint (none) -> Capacitor_SMD:C_0603_1608Metric_Pad1.08x0.95mm_HandSolder
- C26: value C -> 4.7uF; footprint (none) -> Capacitor_SMD:C_0603_1608Metric_Pad1.08x0.95mm_HandSolder
- D1, D2, D3: footprint (none) -> LED_SMD:LED_0603_1608Metric_Pad1.05x0.95mm_HandSolder
- D9: value LED_ABGR -> LED_ABGR CLMVC-FKA-CLBDGL7LBB79353; footprint (none) -> LED_SMD:LED_Cree-PLCC4_2x2mm_CW
- J1: footprint (none) -> Connector_USB:USB_Micro-B_Molex-105017-0001
- J2, J3: footprint (none) -> filestick-footprints:Lumberg_DIN41524_5pin
- J5: footprint (none) -> Connector_PinHeader_2.54mm:PinHeader_1x08_P2.54mm_Vertical
- J6: footprint (none) -> Connector_PinHeader_2.54mm:PinHeader_1x09_P2.54mm_Vertical
- J7, J9: footprint (none) -> Connector_PinHeader_2.54mm:PinHeader_1x02_P2.54mm_Vertical
- J8: footprint (none) -> Connector_PinHeader_2.54mm:PinHeader_2x08_P2.54mm_Vertical
- R1, R11, R12, R13, R14, R2, R24, R29, R3, R4: footprint (none) -> Resistor_SMD:R_0603_1608Metric_Pad0.98x0.95mm_HandSolder
- R5, R6: value R -> 560; footprint (none) -> Resistor_SMD:R_0603_1608Metric_Pad0.98x0.95mm_HandSolder
- TP1, TP2, TP3: footprint (none) -> Connector_PinHeader_2.54mm:PinHeader_1x01_P2.54mm_Horizontal
Connections:
- net +3V3: now also J4.4 (VDD), R35.1; no longer C25.1, D9.1 (A)
- net GND: now also J4.11 (SHIELD), J4.6 (VSS), J4.9 (DET_B)
- net SD_CS: now also J4.2 (DAT3/CD)
- net SD_MISO: now also J4.7 (DAT0)
- net SD_MOSI: now also J4.3 (CMD)
- net SD_SCK: now also J4.5 (CLK)
- net /SD_DETECT: now also J4.10 (DET_A)
- new net: C25.1, D9.1 (A), R35.2
Other:
- moved on the sheet: C25, D9

Commit message: Distribute components on the PCB
Parts:
- C19, C20: footprint Capacitor_SMD:C_0805_2012Metric_Pad1.18x1.45mm_HandSolder -> Capacitor_SMD:C_0603_1608Metric_Pad1.08x0.95mm_HandSolder
- FB1: footprint (none) -> Inductor_SMD:L_0603_1608Metric_Pad1.05x0.95mm_HandSolder
- TP1, TP2, TP3: footprint Connector_PinHeader_2.54mm:PinHeader_1x01_P2.54mm_Horizontal -> Connector_PinHeader_2.54mm:PinHeader_1x01_P2.54mm_Vertical
Connections:
- net SD_CS: now also U1.45 (IOB_5b); no longer U1.48 (IOB_4a)
- net SD_MISO: now also U1.48 (IOB_4a); no longer U1.45 (IOB_5b)
- net SD_MOSI: now also U1.46 (IOB_0a); no longer U1.47 (IOB_2a)
- net SD_SCK: now also U1.47 (IOB_2a); no longer U1.46 (IOB_0a)
Changed lines of the file:
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@@
 	)
 	(junction
-		(at 254 40.64)
-		(diameter 0)
-		(color 0 0 0 0)
-	)
-	(junction
 		(at 317.5 311.15)
 		(diameter 0)
@@
 	)
 	(junction
+		(at 254 40.64)
+		(diameter 0)
+		(color 0 0 0 0)
+	)
+	(junction
 		(at 63.5 251.46)
 		(diameter 0)
@@
 	(wire
 		(pts
+			(xy 254 40.64) (xy 259.08 40.64)
+		)
+		(stroke
+			(width 0)
+			(type default)
+		)
+	)
+	(wire
+		(pts
 			(xy 52.07 140.97) (xy 77.47 140.97)
 		)
@@
 	(wire
 		(pts
+			(xy 157.48 45.72) (xy 170.18 45.72)
+		)
+		(stroke
+			(width 0)
+			(type default)
+		)
+	)
+	(wire
+		(pts
 			(xy 143.51 162.56) (xy 158.75 162.56)
 		)
@@
 	(wire
 		(pts
-			(xy 157.48 45.72) (xy 170.18 45.72)
-		)
-		(stroke
-			(width 0)
-			(type default)
-		)
-	)
-	(wire
-		(pts
 			(xy 281.94 226.06) (xy 307.34 226.06)
 		)
@@
 	(wire
 		(pts
-			(xy 254 40.64) (xy 259.08 40.64)
-		)
-		(stroke
-			(width 0)
-			(type default)
-		)
-	)
-	(wire
-		(pts
 			(xy 486.41 335.28) (xy 486.41 322.58)
 		)
@@
 		)
 	)
-	(label "SD_CS"
-		(at 157.48 50.8 0)
-		(fields_autoplaced yes)
-		(effects
-			(font
-				(size 1.27 1.27)
-			)
-			(justify left bottom)
-		)
-	)
 	(label "UART_TX"
 		(at 127 241.3 0)
@@
 		)
 	)
+	(label "SD_MOSI"
+		(at 157.48 43.18 0)
+		(fields_autoplaced yes)
+		(effects
+			(font
+				(size 1.27 1.27)
+			)
+			(justify left bottom)
+		)
+	)
 	(label "GPIO_13"
 		(at 180.34 157.48 0)
@@
 	)
 	(label "SD_CS"
+		(at 157.48 53.34 0)
+		(fields_autoplaced yes)
+		(effects
+			(font
+				(size 1.27 1.27)
+			)
+			(justify left bottom)
+		)
+	)
+	(label "SD_CS"
 		(at 474.98 50.8 0)
 		(fields_autoplaced yes)
@@
 		)
 	)
-	(label "SD_MOSI"
-		(at 157.48 45.72 0)
-		(fields_autoplaced yes)
-		(effects
-			(font
-				(size 1.27 1.27)
-			)
-			(justify left bottom)
-		)
-	)
 	(label "GPIO_18"
 		(at 58.42 66.04 0)
@@
 		)
 	)
-	(label "SD_SCK"
-		(at 157.48 43.18 0)
-		(fields_autoplaced yes)
-		(effects
-			(font
-				(size 1.27 1.27)
-			)
-			(justify left bottom)
-		)
-	)
 	(label "GPIO_26"
 		(at 180.34 162.56 0)
@@
 		)
 	)
+	(label "SD_SCK"
+		(at 157.48 45.72 0)
+		(fields_autoplaced yes)
+		(effects
+			(font
+				(size 1.27 1.27)
+			)
+			(justify left bottom)
+		)
+	)
 	(label "DATA-"
 		(at 551.18 335.28 0)
@@
 		)
 	)
-	(label "SD_MISO"
-		(at 157.48 53.34 0)
+	(label "USBD_P"
+		(at 43.18 246.38 0)
 		(fields_autoplaced yes)
 		(effects
 			(font
 				(size 1.27 1.27)
+				(italic yes)
 			)
 			(justify left bottom)
 		)
 	)
-	(label "USBD_P"
-		(at 43.18 246.38 0)
+	(label "SD_MISO"
+		(at 157.48 50.8 0)
 		(fields_autoplaced yes)
 		(effects
 			(font
 				(size 1.27 1.27)
-				(italic yes)
 			)
 			(justify left bottom)
@@
 			)
 		)
-		(property "Footprint" "Capacitor_SMD:C_0805_2012Metric_Pad1.18x1.45mm_HandSolder"
+		(property "Footprint" "Capacitor_SMD:C_0603_1608Metric_Pad1.08x0.95mm_HandSolder"
 			(at 322.2752 40.64 0)
 			(effects
@@
 			)
 		)
-		(property "Footprint" "Capacitor_SMD:C_0805_2012Metric_Pad1.18x1.45mm_HandSolder"
+		(property "Footprint" "Capacitor_SMD:C_0603_1608Metric_Pad1.08x0.95mm_HandSolder"
 			(at 322.2752 86.36 0)
 			(effects
@@
 			)
 		)
-		(property "Footprint" "Connector_PinHeader_2.54mm:PinHeader_1x01_P2.54mm_Horizontal"
+		(property "Footprint" "Connector_PinHeader_2.54mm:PinHeader_1x01_P2.54mm_Vertical"
 			(at 322.58 302.26 0)
 			(effects
@@
 			)
 		)
-		(property "Footprint" ""
+		(property "Footprint" "Inductor_SMD:L_0603_1608Metric_Pad1.05x0.95mm_HandSolder"
 			(at 57.15 231.648 90)
 			(effects
@@
 			)
 		)
-		(property "Footprint" "Connector_PinHeader_2.54mm:PinHeader_1x01_P2.54mm_Horizontal"
+		(property "Footprint" "Connector_PinHeader_2.54mm:PinHeader_1x01_P2.54mm_Vertical"
 			(at 519.43 280.67 0)
 			(effects
@@
 			)
 		)
-		(property "Footprint" "Connector_PinHeader_2.54mm:PinHeader_1x01_P2.54mm_Horizontal"
+		(property "Footprint" "Connector_PinHeader_2.54mm:PinHeader_1x01_P2.54mm_Vertical"
 			(at 394.97 322.58 0)
 			(effects

Commit message: Fix econet socket on schematic and route econet front end
Connections:
- net DATA+: now also J3.1; no longer J3.4
- net DATA-: now also J3.4; no longer J3.1
Changed lines of the file:
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@@
 	(wire
 		(pts
+			(xy 309.88 231.14) (xy 309.88 240.03)
+		)
+		(stroke
+			(width 0)
+			(type default)
+		)
+	)
+	(wire
+		(pts
 			(xy 276.86 365.76) (xy 297.18 365.76)
 		)
@@
 	(wire
 		(pts
+			(xy 312.42 226.06) (xy 312.42 242.57)
+		)
+		(stroke
+			(width 0)
+			(type default)
+		)
+	)
+	(wire
+		(pts
 			(xy 58.42 48.26) (xy 76.2 48.26)
 		)
@@
 	(wire
 		(pts
-			(xy 307.34 226.06) (xy 307.34 240.03)
-		)
-		(stroke
-			(width 0)
-			(type default)
-		)
-	)
-	(wire
-		(pts
 			(xy 210.82 34.29) (xy 210.82 35.56)
 		)
@@
 	(wire
 		(pts
-			(xy 307.34 240.03) (xy 304.8 240.03)
+			(xy 304.8 240.03) (xy 309.88 240.03)
 		)
 		(stroke
@@
 	(wire
 		(pts
-			(xy 309.88 242.57) (xy 304.8 242.57)
+			(xy 304.8 242.57) (xy 312.42 242.57)
 		)
 		(stroke
@@
 	(wire
 		(pts
-			(xy 281.94 226.06) (xy 307.34 226.06)
+			(xy 281.94 226.06) (xy 312.42 226.06)
 		)
 		(stroke
@@
 		)
 		(stroke
-			(width 0)
-			(type default)
-		)
-	)
-	(wire
-		(pts
-			(xy 309.88 231.14) (xy 309.88 242.57)
-		)
-		(stroke

Commit message: Improve fpga pin assignments
Connections:
- net COLLISION_DETECT: now also U1.18 (IOB_31b); no longer U1.32 (IOT_43a)
- net COLLISION_REF_PWM: now also U1.13 (IOB_24a); no longer U1.31 (IOT_42b)
- net ECONET_CLKEN: now also U1.6 (IOB_13b); no longer U1.38 (IOT_50b)
- net ECONET_CLKIO: now also U1.43 (IOT_49a), U1.44 (IOB_3b_G6); no longer U1.34 (IOT_44b), U1.35 (IOT_46b_G0)
- net ECONET_RECEIVING: now also U1.19 (IOB_29b); no longer U1.27 (IOT_38b)
- net ECONET_RX: now also U1.11 (IOB_20a); no longer U1.43 (IOT_49a)
- net ECONET_TERM_EN: now also U1.12 (IOB_22a); no longer U1.28 (IOT_41a)
- net ECONET_TX: now also U1.9 (IOB_16a); no longer U1.36 (IOT_48b)
- net ECONET_TX_ENABLE: now also U1.10 (IOB_18a); no longer U1.42 (IOT_51a)
- net GPIO_21: now also J8.12 (Pin_12); no longer J8.9 (Pin_9)
- net GPIO_26: now also J8.9 (Pin_9); no longer J8.10 (Pin_10)
- net GPIO_37: now also J8.1 (Pin_1); no longer J8.11 (Pin_11)
- net UART_RX: now also U1.38 (IOT_50b); no longer U1.25 (IOT_36b)
- net UART_TX: now also U1.42 (IOT_51a); no longer U1.23 (IOT_37a)
- net GPIO_10 renamed GPIO_35
- net GPIO_35: now also U1.35 (IOT_46b_G0); no longer U1.10 (IOB_18a)
- net GPIO_11 renamed GPIO_34
- net GPIO_34: now also U1.34 (IOT_44b); no longer U1.11 (IOB_20a)
- net GPIO_12 renamed GPIO_32
- net GPIO_32: now also U1.32 (IOT_43a); no longer U1.12 (IOB_22a)
- net GPIO_13 renamed GPIO_31
- net GPIO_31: now also U1.31 (IOT_42b); no longer U1.13 (IOB_24a)
- net GPIO_18 renamed GPIO_28
- net GPIO_28: now also U1.28 (IOT_41a); no longer U1.18 (IOB_31b)
- net GPIO_19 renamed GPIO_27
- net GPIO_27: now also U1.27 (IOT_38b); no longer U1.19 (IOB_29b)
- removed net GPIO_44: J8.12 (Pin_12), U1.44 (IOB_3b_G6)
- removed net GPIO_6: J8.1 (Pin_1), U1.6 (IOB_13b)
- net GPIO_9 renamed GPIO_36
- net GPIO_36: now also U1.36 (IOT_48b); no longer U1.9 (IOB_16a)
- new net GPIO_23: J8.11 (Pin_11), U1.23 (IOT_37a)
- new net GPIO_25: J8.10 (Pin_10), U1.25 (IOT_36b)
Other:
- note added: "Note: Input"
- note added: "Note: output"

Commit message: Route the rest of the PCB
Parts:
- added C14: 100nF, Capacitor_SMD:C_0603_1608Metric_Pad1.08x0.95mm_HandSolder, symbol Device:C
- added SW1: SW_Push, Button_Switch_SMD:SW_SPST_PTS645, symbol Switch:SW_Push
- renumbered C11 to C1, C27 to C10, C16 to C11, C25 to C12, C4 to C13, C5 to C15, C15 to C16, C14 to C17, C29 to C18, C26 to C19, C1 to C2, C6 to C20, C24 to C21, C8 to C22, C20 to C23, C23 to C24, C17 to C25, C19 to C26, C12 to C27, C10 to C28, C22 to C29, C18 to C30, C7 to C31, C21 to C32, C9 to C33, C2 to C4, C13 to C5, C28 to C6, C30 to C7, C31 to C8, C32 to C9, D11 to D1, D7 to D10, D1 to D11, D8 to D12, D12 to D2, D10 to D3, D9 to D4, D3 to D5, D2 to D6, D4 to D7, D5 to D8, D6 to D9, J2 to J1, J4 to J2, J1 to J3, J3 to J4, J6 to J5, J7 to J6, J9 to J7, J5 to J9, Q4 to Q1, Q5 to Q2, Q2 to Q4, Q1 to Q5, R34 to R1, R33 to R10, R16 to R11, R25 to R12, R18 to R13, R27 to R14, R26 to R15, R4 to R16, R35 to R17, R6 to R18, R5 to R19, R31 to R2, R22 to R20, R8 to R21, R23 to R22, R15 to R23, R9 to R24, R20 to R25, R10 to R26, R17 to R27, R19 to R28, R12 to R29, R7 to R3, R11 to R30, R13 to R31, R14 to R32, R1 to R33, R24 to R34, R21 to R35, R29 to R4, R3 to R5, R2 to R6, R32 to R7, R30 to R8, R28 to R9, TP2 to TP1, TP3 to TP2, TP1 to TP3, U4 to U1, U3 to U2, U8 to U3, U1 to U4, U2 to U5, U5 to U6, U6 to U8
Connections:
- net +1V2: now also C14.2
- net +3V3: now also C16.1; no longer C16.2
- net ECONET_CLKIO: no longer U4.43 (IOT_49a)
- net GND: now also C16.2, C14.1, SW1.1; no longer C16.1, J8.14 (Pin_14)
- net GPIO_21: now also J8.14 (Pin_14); no longer J8.12 (Pin_12)
- net GPIO_25: now also J8.12 (Pin_12); no longer J8.10 (Pin_10)
- net GPIO_27: now also J8.10 (Pin_10); no longer J8.8 (Pin_8)
- net GPIO_31: now also J8.8 (Pin_8); no longer J8.6 (Pin_6)
- net GPIO_34: now also J8.6 (Pin_6); no longer J8.4 (Pin_4)
- net GPIO_36: now also J8.4 (Pin_4); no longer J8.2 (Pin_2)
- net UART_RX: now also U4.37 (IOT_45a_G1); no longer U4.38 (IOT_50b)
- net UART_TX: now also U4.38 (IOT_50b); no longer U4.42 (IOT_51a)
- net /CRESET: now also SW1.2
- net USB+: now reaches R5.2, U5.8 (USBDP)
- net USB-: now reaches R6.2, U5.9 (USBDM)
- net GPIO_37 renamed GPIO_42
- net GPIO_42: now also U4.42 (IOT_51a); no longer U4.37 (IOT_45a_G1)
- new net GPIO_43: J8.2 (Pin_2), U4.43 (IOT_49a)
Other:
- note removed: "Note: Input"
- note removed: "Note: output"
- moved on the sheet: C16

Commit message: Update kicad files to v9, turn micro-sd card slot the right way
Parts:
- U1, U2: footprint Package_SO:SO-8_5.3x6.2mm_P1.27mm -> Package_SO:SOIC-8_5.3x6.2mm_P1.27mm
Connections:
- net SD_CS: now also J5.5 (Pin_5), U4.2 (IOB_6a); no longer J5.1 (Pin_1), U4.45 (IOB_5b)
- net SD_MISO: now also J5.2 (Pin_2), U4.46 (IOB_0a); no longer J5.4 (Pin_4), U4.48 (IOB_4a)
- net SD_MOSI: now also J5.4 (Pin_4), U4.48 (IOB_4a); no longer J5.2 (Pin_2), U4.46 (IOB_0a)
- net /SD_DETECT: now also J5.1 (Pin_1), U4.45 (IOB_5b); no longer J5.5 (Pin_5), U4.2 (IOB_6a)
Other:
- moved on the sheet: C27, C28
